Commit message: update the ft sensor

File: universal_robot/ur_e_description/urdf/common.gazebo.xacro (robot description, xacro)
@@ -22,3 +22,13 @@
 -->
   </gazebo>
+  <gazebo reference="wrist_3_joint">
+     <provideFeedback>true</provideFeedback>
+  </gazebo>
+  <gazebo>
+    <plugin name="wrench" filename="libgazebo_ros_ft_sensor.so">
+      <updateRate>100.0</updateRate>
+      <topicName>wrench</topicName>
+      <jointName>wrist_3_joint</jointName>
+    </plugin>
+</gazebo>
 </robot>

File: universal_robot/ur_e_description/urdf/ur.transmission.xacro (robot description, xacro)
@@ -6,4 +6,5 @@
       <joint name="${prefix}shoulder_pan_joint">
         <hardwareInterface>hardware_interface/PositionJointInterface</hardwareInterface>
+        <!-- <hardwareInterface>hardware_interface/EffortJointInterface</hardwareInterface> -->
       </joint>
       <actuator name="${prefix}shoulder_pan_motor">
@@ -15,4 +16,5 @@
       <joint name="${prefix}shoulder_lift_joint">
         <hardwareInterface>hardware_interface/PositionJointInterface</hardwareInterface>
+        <!-- <hardwareInterface>hardware_interface/EffortJointInterface</hardwareInterface> -->
       </joint>
       <actuator name="${prefix}shoulder_lift_motor">
@@ -24,4 +26,5 @@
       <joint name="${prefix}elbow_joint">
         <hardwareInterface>hardware_interface/PositionJointInterface</hardwareInterface>
+        <!-- <hardwareInterface>hardware_interface/EffortJointInterface</hardwareInterface> -->
       </joint>
       <actuator name="${prefix}elbow_motor">
@@ -33,4 +36,5 @@
       <joint name="${prefix}wrist_1_joint">
         <hardwareInterface>hardware_interface/PositionJointInterface</hardwareInterface>
+        <!-- <hardwareInterface>hardware_interface/EffortJointInterface</hardwareInterface> -->
       </joint>
       <actuator name="${prefix}wrist_1_motor">
@@ -42,4 +46,5 @@
       <joint name="${prefix}wrist_2_joint">
         <hardwareInterface>hardware_interface/PositionJointInterface</hardwareInterface>
+        <!-- <hardwareInterface>hardware_interface/EffortJointInterface</hardwareInterface> -->
       </joint>
       <actuator name="${prefix}wrist_2_motor">
@@ -51,4 +56,5 @@
       <joint name="${prefix}wrist_3_joint">
         <hardwareInterface>hardware_interface/PositionJointInterface</hardwareInterface>
+        <!-- <hardwareInterface>hardware_interface/EffortJointInterface</hardwareInterface> -->
       </joint>
       <actuator name="${prefix}wrist_3_motor">

File: universal_robot/ur_e_description/urdf/ur5e.urdf.xacro (robot description, xacro)
@@ -350,4 +350,20 @@
       <child link="${prefix}tool0"/>
     </joint>
+    <!-- wrench sensor -->
+    <joint name="wrench_sensor_joint" type="revolute">
+      <parent link="${prefix}ee_link" />
+      <child link="${prefix}wrench_link" />
+      <axis xyz="0 0 1" />
+      <origin xyz="0.0 0.0 0.0" rpy="0.0 0.0 ${pi/2.0}" />
+      <limit velocity="6.5" effort="1000" lower="0" upper="0" />
+    </joint>
+    <link name="${prefix}wrench_link">
+      <collision>
+        <geometry>
+          <box size="0.01 0.01 0.01"/>
+        </geometry>
+        <origin rpy="0 0 0" xyz="-0.01 0 0"/>
+      </collision>
+    </link>
   </xacro:macro>
 </robot>
